Commit message: add_model

File: src/robot_model/urdf/crs_a465.urdf (robot description, URDF)
Before this commit: robot crs_a465, 7 links, 6 joints
Links:
- added link end_effector; collision mesh filename=meshes/herramienta.stl scale=1 1 1; visual mesh filename=meshes/herramienta.stl scale=1 1 1
- added link hoop_adapter_link; collision mesh filename=meshes/CRS_adapter.stl scale=0.001 0.001 0.001; visual mesh filename=meshes/CRS_adapter.stl scale=0.001 0.001 0.001
- added link hoop_link; collision mesh filename=meshes/Hoop.stl scale=0.001 0.001 0.001; visual mesh filename=meshes/Hoop.stl scale=0.001 0.001 0.001
- link base_link: geometry collision mesh filename=meshes/base_estatica.stl scale=1 1 1; visual mesh filename=meshes/base_estatica.stl scale=1 1 1
- link link1: geometry collision mesh filename=meshes/codos_por_fuera.stl scale=1 1 1; visual mesh filename=meshes/codos_por_fuera.stl scale=1 1 1
- link link2: geometry collision mesh filename=meshes/brazo1.stl scale=1 1 1; visual mesh filename=meshes/brazo1.stl scale=1 1 1
- link link3: geometry collision mesh filename=meshes/anexo_brazo2.stl scale=1 1 1; visual mesh filename=meshes/anexo_brazo2.stl scale=1 1 1
- link link4: geometry collision mesh filename=meshes/brazo2_sin_herramienta.stl scale=1 1 1; visual mesh filename=meshes/brazo2_sin_herramienta.stl scale=1 1 1
- link tool_link: geometry collision mesh filename=meshes/union_herramienta.stl scale=1 1 1; visual mesh filename=meshes/union_herramienta.stl scale=1 1 1
Joints:
- added joint joint6: type revolute, parent tool_link, child end_effector, origin xyz=0 0 0 rpy=1.57079632679 0 0, axis 0 0 1, limit lower=-3.142 upper=3.142 effort=10 velocity=3
- added joint joint7: type fixed, parent end_effector, child hoop_adapter_link, origin xyz=0 0 0 rpy=0 0 0
- added joint joint8: type fixed, parent hoop_adapter_link, child hoop_link, origin xyz=0 0 0 rpy=0 0 0
- joint joint4: axis 0 0 1 -> 0 0 -1
- joint joint5: axis 0 0 1 -> 0 0 -1

Commit message: fix_collision

File: src/robot_model/urdf/crs_a465.urdf (robot description, URDF)
Before this commit: robot crs_a465, 10 links, 9 joints
Joints:
- joint joint4: axis 0 0 -1 -> 0 0 1
